File: CM4_GPIO.kicad_sch (KiCad schematic)
At the start: 28 parts, among them J1 Conn_01x03, J2 Conn_02x07_Odd_Even, J3 Conn_01x03, J7 Micro_SD_Card_Det, J8 THD-20-R, J9 THD-02-R, U1 TPD4EUSB30, U18 RT9742GGJ5, U2 TPD4EUSB30, U3 MagJack-A70-112-331N126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

Commit message: Removing unneeded items
Connections:
- net TV_OUT: no longer names the net of J2.11 (Pin_11)
